File: E-PIX/E-PIX.kicad_pcb (KiCad board)
At the start: 6 copper layers, 40.1 x 45 mm, 69 parts, among them J1 USB_C_Receptacle_USB2.0, J2 DM3AT-SF-PEJM5, Q1 AO3401A, Q2 2SC4213, Q3 2SC4213, Q4 BSS138, Q5 BSS138, SW1 SW_Push, SW2 SW_Push, U10 ESP32-S3-WROOM-1, U2 NJM7805SDL1, U3 AZ1117-3.3, U4 BTS6142D, U5 Conn_03x02, U6 Conn_03x04, U7 U7, U8 U8, U9 FT231XS

Commit message: fix sketch error
Parts:
- removed the D4 at (147.9, 83.4)
- removed the Q1 at (134.3, 83.6)
- removed the R1 at (157.8, 107.2)
- removed the R3 at (130.5, 82.7)
- removed the R4 at (147.8, 87.3)
- added C6: 0.1u, Capacitor_SMD:C_0603_1608Metric, F.Cu at (119.0, 95.5)
- added R7: 2.2k, Resistor_SMD:R_0805_2012Metric, F.Cu at (114.8, 95.7)
- added R8: 2.2k, Resistor_SMD:R_0805_2012Metric, F.Cu at (114.8, 98.6)
- added R9: 10k, Resistor_SMD:R_0603_1608Metric, F.Cu at (119.0, 98.0)
- C11: renamed from C1; value 10u/50V/2012 -> 10u/50V/3216; footprint Capacitor_SMD:C_0805_2012Metric -> Capacitor_SMD:C_1206_3216Metric
- R1: renamed from R19; footprint Resistor_SMD:R_0603_1608Metric -> Resistor_SMD:R_0805_2012Metric
- R11: renamed from R6; footprint Resistor_SMD:R_0603_1608Metric -> Resistor_SMD:R_0805_2012Metric
- R12: renamed from R9; footprint Resistor_SMD:R_0603_1608Metric -> Resistor_SMD:R_0805_2012Metric
- R16, R17: footprint Resistor_SMD:R_0603_1608Metric -> Resistor_SMD:R_0805_2012Metric
- R18: renamed from R20; footprint Resistor_SMD:R_0603_1608Metric -> Resistor_SMD:R_0805_2012Metric
- R19: renamed from R21; footprint Resistor_SMD:R_0603_1608Metric -> Resistor_SMD:R_0805_2012Metric
- R2: renamed from R7; footprint Resistor_SMD:R_0603_1608Metric -> Resistor_SMD:R_0805_2012Metric
- R21: renamed from R14; footprint Resistor_SMD:R_0603_1608Metric -> Resistor_SMD:R_0805_2012Metric
- R3: renamed from R8; footprint Resistor_SMD:R_0603_1608Metric -> Resistor_SMD:R_0805_2012Metric
- U4: renamed from U2; value NJM7805SDL1 -> LM78M05RS
- U5: renamed from U7; value U7 -> TC7WH241FK
- U6: renamed from U8; value U8 -> TC7WH241FK
- moved Q3 0.39 mm to (144.8, 103.6)
- moved R18 0.35 mm to (155.5, 103.5)
- moved R17 0.12 mm to (144.9, 105.8)
- renumbered C11 to C1, C1 to C10, C5 to C12, C6 to C13, C3 to C2, C12 to C3, C7 to C4, C8 to C5, C2 to C7, C4 to C8, D9 to D1, D5 to D2, D2 to D3, D8 to D4, D1 to D5, D3 to D6, D6 to D8, Q2 to Q1, Q3 to Q2, Q4 to Q3, Q5 to Q4, R15 to R10, R5 to R13, R10 to R14, R18 to R15, R11 to R20, R12 to R4, R13 to R5, R2 to R6, SW2 to SW1, SW1 to SW2, U9 to U1, U6 to U10, U10 to U2, U4 to U3, U3 to U7, BNO055 to U8, U5 to U9
Connections:
- D5 pad 2: Net-(D1-A) -> +5V
- R6 pad 1: Net-(U4-IS) -> Net-(U3-IN)
- U1 pad 13: +3V3 -> Net-(U1-3V3OUT)
- U1 pad 14: unconnected-(U9-~{RESET}-Pad14) -> Net-(U1-3V3OUT)
- U1 pad 3: +3V3 -> Net-(U1-3V3OUT)
- U2 pad 13: /TX2 -> /ESP_D-
- U2 pad 14: /RX2 -> /ESP_D+
- U2 pad 15: /EN2 -> /Floating
- U2 pad 16: unconnected-(U10-IO46-Pad16) -> Net-(U2-IO45)
- U2 pad 26: /EN_Power -> Net-(U2-IO45)
- U3 pad 2: Net-(U4-IN) -> Net-(U3-IN)
- U3 pad 4: Net-(U4-IS) -> Net-(U3-IN)
Routing:
- net VSS: track 112.2 -> 88.6 mm, vias 27 -> 25
- net Net-(U4-IN): track 9.86 -> 0.00 mm
- net Net-(U3-IN): track 0.00 -> 8.66 mm
- net /EN_Power: track 8.15 -> 0.00 mm, vias 2 -> 0
- net Net-(U1-3V3OUT): track 0.00 -> 7.21 mm, vias 0 -> 2
- net Net-(U4-IS): track 6.38 -> 0.00 mm
- net +5V: track 77.8 -> 83.2 mm
- net Net-(D4-K) (its old number): track 5.28 -> 0.00 mm
- net +3V3: track 177.9 -> 174.0 mm, vias 24 -> 22
- net Net-(D1-A): track 3.76 -> 0.00 mm
- net /ICS2_5V: track 22.6 -> 23.2 mm
- net GND: vias 159 -> 157

Commit message: correct all errors. waiting for check. (order tomorrow)
Parts:
- C6, R7, R8, R9: moved to B.Cu
- R1, R21: value 100 -> 1k
- R2, R3: value 5.1k -> 4.7k
- R4, R5: value 27 -> 21
- moved C6 40.1 mm to (157.2, 83.0), turned to 90 degrees
- moved R9 33.7 mm to (152.7, 97.5)
- moved R8 24.9 mm to (138.7, 91.7), turned to 180 degrees
- moved R7 24.7 mm to (138.7, 89.8), turned to 180 degrees
- moved D2 19.2 mm to (151.4, 100.0)
- moved R10 17.3 mm to (140.0, 85.4)
- moved U5 4.46 mm to (132.4, 99.0)
- moved U6 4.43 mm to (128.0, 98.9)
- moved R1 3.90 mm to (147.9, 87.3)
- moved R21 2.71 mm to (142.9, 87.3), turned to 0 degrees
- moved D1 1.25 mm to (146.7, 83.4)
- moved D7 1.25 mm to (144.1, 83.4)
- moved D4 0.63 mm to (127.2, 118.4)
- turned U8 to 0 degrees
Connections:
- net /Floating renamed /JTAG
- Q3 pad 2: /ICS1_3V3 -> /ICS2_3V3
- Q3 pad 3: /ICS1_5V -> /ICS2_5V
- Q4 pad 2: /ICS2_3V3 -> /ICS1_3V3
- Q4 pad 3: /ICS2_5V -> /ICS1_5V
- R16 pad 2: /ICS1_3V3 -> /ICS2_3V3
- R17 pad 2: /ICS1_5V -> /ICS2_5V
- R18 pad 2: /ICS2_3V3 -> /ICS1_3V3
- R19 pad 2: /ICS2_5V -> /ICS1_5V
- R7 pad 2: /SDA -> /SCL
- R8 pad 2: /SCL -> /SDA
- R9 pad 1: Net-(U2-IO45) -> /SPI_vol
- U10 pad 3: /ICS1_5V -> /ICS2_5V
- U2 pad 12: /SDA -> /EN1
- U2 pad 16: Net-(U2-IO45) -> /ROM_print
- U2 pad 17: /SCL -> /BNO_RST
- U2 pad 26: Net-(U2-IO45) -> /SPI_vol
- U2 pad 4: unconnected-(U2-IO4-Pad4) -> /SCL
- U2 pad 5: unconnected-(U2-IO5-Pad5) -> /SDA
- U2 pad 7: /BNO_RST -> /RX2
- U2 pad 8: unconnected-(U2-IO15-Pad8) -> /TX2
- U2 pad 9: /EN1 -> /EN2
- U9 pad 3: /ICS2_5V -> /ICS1_5V
Routing:
- net +3V3: track 174.0 -> 127.8 mm, vias 22 -> 24
- net Net-(D2-A): track 39.2 -> 20.7 mm, vias 2 -> 1
- net /SDA: track 6.40 -> 20.5 mm
- net +5V: track 83.2 -> 96.9 mm
- net Net-(U1-3V3OUT): track 7.21 -> 16.6 mm
- net /RX2: track 4.96 -> 13.4 mm
- net /SCL: track 12.8 -> 20.9 mm
- net /TX2: track 4.20 -> 11.9 mm
- net /EN1: track 15.0 -> 10.2 mm
- net /RX1: track 10.9 -> 6.35 mm
- net /ICS1_3V3: track 22.2 -> 26.7 mm
- net /SPI_vol: track 0.00 -> 4.36 mm, vias 0 -> 1
- net /EN2: track 11.1 -> 15.3 mm
- net /BNO_RST: track 18.6 -> 14.4 mm
- net /ICS2_3V3: track 26.0 -> 22.2 mm
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Other:
- board text added: "GND/VSS/ICS2"
- board text added: "ICS1/VSS/GND"
- board text removed: "GND/VSS/ICS1"
- board text removed: "ICS2/VSS/GND"
- board text removed: "VSS"

Commit message: go thorough last check. order
Parts:
- R13: renamed from R18; footprint Resistor_SMD:R_0805_2012Metric -> Resistor_SMD:R_0603_1608Metric
- R14: renamed from R19; footprint Resistor_SMD:R_0805_2012Metric -> Resistor_SMD:R_0603_1608Metric
- R20: renamed from R16; footprint Resistor_SMD:R_0805_2012Metric -> Resistor_SMD:R_0603_1608Metric
- R21: renamed from R17; footprint Resistor_SMD:R_0805_2012Metric -> Resistor_SMD:R_0603_1608Metric
- U7: renamed from U6; value TC7WH241FK -> U7
- U8: renamed from U5; value TC7WH241FK -> U8
- moved U7 0.13 mm to (128.0, 99.0)
- renumbered C11 to C1, C9 to C10, C10 to C11, C1 to C12, C3 to C13, C7 to C2, C2 to C3, C8 to C4, C12 to C5, C13 to C6, C4 to C7, C5 to C8, C6 to C9, D5 to D1, D3 to D2, D6 to D3, D2 to D4, D8 to D5, D7 to D6, D4 to D7, D1 to D8, Q4 to Q3, Q3 to Q4, R6 to R1, R5 to R10, R21 to R11, R10 to R12, R7 to R16, R9 to R17, R8 to R18, R1 to R19, R13 to R2, R11 to R3, R2 to R4, R3 to R5, R12 to R6, R14 to R7, R20 to R8, R4 to R9, SW2 to SW1, SW1 to SW2, U8 to U1, U2 to U10, U4 to U2, U7 to U3, U3 to U4, U9 to U5, U10 to U6, U1 to U9
Routing:
- net +3V3: track 127.8 -> 129.6 mm
- net /EN2: track 15.3 -> 16.0 mm
Other:
- board text added: "v1 2026/01/23"
- board text removed: "v0 2025/12/15"
