File: E-PIX/E-PIX.kicad_sch (KiCad schematic)
At the start: 65 parts, among them J1 USB_C_Receptacle_USB2.0, J2 DM3AT-SF-PEJM5, Q1 AO3401A, Q2 2SC4213, Q3 2SC4213, Q4 BSS138, Q5 BSS138, SW1 SW_Push, SW2 SW_Push, U10 ESP32-S3-WROOM-1, U2 NJM7805SDL1, U3 AZ1117-3.3, U4 BTS6142D, U5 Conn_03x02, U6 Conn_03x04, U7 TC7WH241FK, U8 TC7WH241FK, U9 FT231XS

Commit message: fix sketch error
Parts:
- removed D4: LED, LED_SMD:LED_0603_1608Metric, symbol Device:LED
- removed Q1: AO3401A, Package_TO_SOT_SMD:SOT-23, symbol Transistor_FET:AO3401A
- removed R1: 10k, Resistor_SMD:R_0603_1608Metric, symbol Device:R_Small
- removed R3: 4.7, Resistor_SMD:R_0603_1608Metric, symbol Device:R
- removed R4: 100, Resistor_SMD:R_0603_1608Metric, symbol Device:R
- added C6: 0.1u, Capacitor_SMD:C_0603_1608Metric, symbol Device:C
- added R7, R8: 2.2k, Resistor_SMD:R_0805_2012Metric, symbol Device:R
- added R9: 10k, Resistor_SMD:R_0603_1608Metric, symbol Device:R
- C11: renamed from C1; value 10u/50V/2012 -> 10u/50V/3216; footprint Capacitor_SMD:C_0805_2012Metric -> Capacitor_SMD:C_1206_3216Metric
- R1: renamed from R19; footprint Resistor_SMD:R_0603_1608Metric -> Resistor_SMD:R_0805_2012Metric
- R11: renamed from R6; footprint Resistor_SMD:R_0603_1608Metric -> Resistor_SMD:R_0805_2012Metric
- R12: renamed from R9; footprint Resistor_SMD:R_0603_1608Metric -> Resistor_SMD:R_0805_2012Metric
- R16, R17: footprint Resistor_SMD:R_0603_1608Metric -> Resistor_SMD:R_0805_2012Metric
- R18: renamed from R20; footprint Resistor_SMD:R_0603_1608Metric -> Resistor_SMD:R_0805_2012Metric
- R19: renamed from R21; footprint Resistor_SMD:R_0603_1608Metric -> Resistor_SMD:R_0805_2012Metric
- R2: renamed from R7; footprint Resistor_SMD:R_0603_1608Metric -> Resistor_SMD:R_0805_2012Metric
- R21: renamed from R14; footprint Resistor_SMD:R_0603_1608Metric -> Resistor_SMD:R_0805_2012Metric
- R3: renamed from R8; footprint Resistor_SMD:R_0603_1608Metric -> Resistor_SMD:R_0805_2012Metric
- U4: renamed from U2; value NJM7805SDL1 -> LM78M05RS
- renumbered C11 to C1, C5 to C12, C6 to C13, C3 to C2, C12 to C3, C7 to C4, C8 to C5, C2 to C7, C4 to C8, D9 to D1, D5 to D2, D2 to D3, D8 to D4, D1 to D5, D3 to D6, D6 to D8, Q2 to Q1, Q3 to Q2, Q4 to Q3, Q5 to Q4, R15 to R10, R5 to R13, R10 to R14, R18 to R15, R11 to R20, R12 to R4, R13 to R5, R2 to R6, SW2 to SW1, SW1 to SW2, U9 to U1, U6 to U10, U10 to U2, U4 to U3, U7 to U5, U8 to U6, U3 to U7, U1 to U8, U5 to U9
Connections:
- net EN_Power is gone; now on an unnamed net: U2.26 (IO45)
- net +3V3: now also R7.1, R8.1; no longer U1.13 (3V3OUT), U1.3 (VCCIO)
- net +5V: now also D5.2 (A)
- net EN2: no longer U2.15 (IO3)
- net GND: now also C6.2, R9.2
- net RX2: no longer U2.14 (USB_D+)
- net SCL: now also R8.2
- net SDA: now also R7.2
- net TX2: no longer U2.13 (USB_D-)
- net at R6.1, U3.4 (IS): now also U3.2 (IN)
- net at U2.16 (IO46): now also R9.1
- net at U1.14 (~{RESET}): now also U1.13 (3V3OUT), U1.3 (VCCIO), C6.1
- new net ESP_D+: U2.14 (USB_D+)
- new net ESP_D-: U2.13 (USB_D-)
- new net Floating: U2.15 (IO3)
- no-connect marks 32 -> 30
Other:
- moved on the sheet: C1, C3, C4, C5, D1, D2, D4, H1, H2, J1, Q3, R1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

Commit message: correct all errors. waiting for check. (order tomorrow)
Parts:
- R1, R21: value 100 -> 1k
- R2, R3: value 5.1k -> 4.7k
- R4, R5: value 27 -> 21
Connections:
- net BNO_RST: now also U2.17 (IO9); no longer U2.7 (IO7)
- net EN1: now also U2.12 (IO8); no longer U2.9 (IO16)
- net EN2: now also U2.9 (IO16)
- net ICS1_3V3: now also Q4.2 (S), R18.2; no longer Q3.2 (S), R16.2
- net ICS1_5V: now also Q4.3 (D), R19.2, U9.3 (ICS); no longer Q3.3 (D), R17.2, U10.3 (ICS)
- net ICS2_3V3: now also Q3.2 (S), R16.2; no longer Q4.2 (S), R18.2
- net ICS2_5V: now also Q3.3 (D), R17.2, U10.3 (ICS); no longer Q4.3 (D), R19.2, U9.3 (ICS)
- net RX2: now also U2.7 (IO7)
- net SCL: now also R7.2, U2.4 (IO4); no longer R8.2, U2.17 (IO9)
- net SDA: now also R8.2, U2.5 (IO5); no longer R7.2, U2.12 (IO8)
- net TX2: now also U2.8 (IO15)
- net SPI_vol: now reaches R9.1, U2.26 (IO45)
- net SPI_vol: no longer U2.16 (IO46)
- net Floating renamed JTAG
- new net ROM_print: U2.16 (IO46)
- no-connect marks 30 -> 27
Other:
- moved on the sheet: C1, C3, D1, R1, R7, R8, R9, U2

Commit message: go thorough last check. order
Parts:
- R13: renamed from R18; footprint Resistor_SMD:R_0805_2012Metric -> Resistor_SMD:R_0603_1608Metric
- R14: renamed from R19; footprint Resistor_SMD:R_0805_2012Metric -> Resistor_SMD:R_0603_1608Metric
- R20: renamed from R16; footprint Resistor_SMD:R_0805_2012Metric -> Resistor_SMD:R_0603_1608Metric
- R21: renamed from R17; footprint Resistor_SMD:R_0805_2012Metric -> Resistor_SMD:R_0603_1608Metric
- renumbered C11 to C1, C9 to C10, C10 to C11, C1 to C12, C3 to C13, C7 to C2, C2 to C3, C8 to C4, C12 to C5, C13 to C6, C4 to C7, C5 to C8, C6 to C9, D5 to D1, D3 to D2, D6 to D3, D2 to D4, D8 to D5, D7 to D6, D4 to D7, D1 to D8, Q4 to Q3, Q3 to Q4, R6 to R1, R5 to R10, R21 to R11, R10 to R12, R7 to R16, R9 to R17, R8 to R18, R1 to R19, R13 to R2, R11 to R3, R2 to R4, R3 to R5, R12 to R6, R14 to R7, R20 to R8, R4 to R9, SW2 to SW1, SW1 to SW2, U8 to U1, U2 to U10, U4 to U2, U7 to U3, U3 to U4, U9 to U5, U10 to U6, U6 to U7, U5 to U8, U1 to U9
Other:
- moved on the sheet: Q3, Q4, R13, R14, R20, R21, U7, U8
